File: switched_power_supply/switched_power_supply.kicad_pcb (KiCad board)
At the start: 2 copper layers, 38 parts, among them IC1 VIPER53ESPTR-E, T1 Transformador_1x2, U1 Viper53, U2 TL431, U3 PC817 Opto

Commit message: Uploading files
Parts:
- T1: footprint Transformer_SMD:Transformer_Wuerth_750315371 -> pci:TRZ 25.010.2
- moved T1 17.6 mm to (236.6, 136.1)

Commit message: aula 17.02
Parts:
- removed C1: Capacitor_Eletrolitico, pci:EEHZT1E331UP
- removed C2b1: Capacitor_Eletrolitico, Capacitor_THT:CP_Radial_D16.0mm_P7.50mm
- D4: value SR5200 -> RFN4RSM2S; footprint Diode_THT:D_DO-201AD_P15.24mm_Horizontal -> Package_TO_SOT_SMD:TO-277A
- moved V1 253.1 mm to (30.4, 31.3), turned to 90 degrees
- moved F1 213.2 mm to (37.9, 30.6)
- moved T1 203.0 mm to (47.3, 62.9)
- moved C3b1 180.2 mm to (44.0, 44.3), turned to 180 degrees
- moved C8 176.4 mm to (44.0, 51.8), turned to 180 degrees
- moved C3 158.4 mm to (51.5, 26.2), turned to 180 degrees
- moved D4 138.7 mm to (106.1, 94.3)
- moved C5 130.0 mm to (102.7, 39.2), turned to -90 degrees
- moved L1 126.0 mm to (81.2, 30.4), turned to 180 degrees
- moved C6 119.6 mm to (145.6, 87.3)
- moved D2 119.6 mm to (143.5, 69.3)
- moved R5 119.6 mm to (140.8, 87.1)
- moved R6 119.6 mm to (140.8, 90.1)
- moved R7 119.6 mm to (140.8, 93.0)
- moved R8 119.6 mm to (140.8, 96.0)
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Routing:
- net /BarP: track 0.00 -> 72.0 mm
- net GND: track 0.00 -> 34.3 mm
- net Net-(D3-K): track 0.00 -> 32.6 mm
- net Net-(C3-Pad2): track 0.00 -> 29.3 mm
- net Net-(C3-Pad1): track 0.00 -> 17.8 mm
- net Net-(D1d2-A): track 0.00 -> 14.7 mm
- net Net-(D1d1-K): track 0.00 -> 14.6 mm
- net Net-(F1-Pad1): track 0.00 -> 7.73 mm
Other:
- board outline added: 80 x 60 mm

Commit message: aula 17.02
Parts:
- moved C5 19.3 mm to (101.9, 58.5)
- moved D1d2 3.43 mm to (87.5, 34.5)
- moved D1d1 3.43 mm to (87.5, 25.5)
- moved D1d3 3.43 mm to (87.5, 30.0)
- moved D1d4 3.43 mm to (87.3, 39.0)
Routing:
- net GND: track 34.3 -> 29.3 mm
- net /BarP: track 72.0 -> 68.4 mm
- net Net-(D3-K): track 32.6 -> 32.1 mm
Changed lines of the file:
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@@
 	(footprint "Diode_THT:D_A-405_P12.70mm_Horizontal"
 		(layer "F.Cu")
-		(at 84.1 30.7)
+		(at 87.45 29.975)
 		(descr "Diode, A-405 series, Axial, Horizontal, pin pitch=12.7mm, , length*diameter=5.2*2.7mm^2, , http://www.diodes.com/_files/packages/A-405.pdf")
 		(tags "Diode A-405 series Axial Horizontal pin pitch 12.7mm  length 5.2mm diameter 2.7mm")
@@
 	(footprint "Diode_THT:D_A-405_P12.70mm_Horizontal"
 		(layer "F.Cu")
-		(at 84.1 35.2)
+		(at 87.45 34.475)
 		(descr "Diode, A-405 series, Axial, Horizontal, pin pitch=12.7mm, , length*diameter=5.2*2.7mm^2, , http://www.diodes.com/_files/packages/A-405.pdf")
 		(tags "Diode A-405 series Axial Horizontal pin pitch 12.7mm  length 5.2mm diameter 2.7mm")
@@
 	(footprint "Diode_THT:D_A-405_P12.70mm_Horizontal"
 		(layer "F.Cu")
-		(at 84.1 26.2)
+		(at 87.45 25.475)
 		(descr "Diode, A-405 series, Axial, Horizontal, pin pitch=12.7mm, , length*diameter=5.2*2.7mm^2, , http://www.diodes.com/_files/packages/A-405.pdf")
 		(tags "Diode A-405 series Axial Horizontal pin pitch 12.7mm  length 5.2mm diameter 2.7mm")
@@
 	(footprint "Diode_THT:D_A-405_P12.70mm_Horizontal"
 		(layer "F.Cu")
-		(at 83.95 39.7)
+		(at 87.3 38.975)
 		(descr "Diode, A-405 series, Axial, Horizontal, pin pitch=12.7mm, , length*diameter=5.2*2.7mm^2, , http://www.diodes.com/_files/packages/A-405.pdf")
 		(tags "Diode A-405 series Axial Horizontal pin pitch 12.7mm  length 5.2mm diameter 2.7mm")
@@
 		(tags "CP Radial series Radial pin pitch 7.50mm  diameter 16mm Electrolytic Capacitor")
 		(property "Reference" "C7"
-			(at 3.75 -9.25 0)
+			(at 7.1 -9.975 0)
 			(layer "F.SilkS")
 			(effects
@@
 	(footprint "Capacitor_THT:C_Rect_L7.0mm_W2.5mm_P5.00mm"
 		(layer "F.Cu")
-		(at 102.7 39.2 -90)
+		(at 101.9 58.45 -90)
 		(descr "C, Rect series, Radial, pin pitch=5.00mm, , length*width=7*2.5mm^2, Capacitor")
 		(tags "C Rect series Radial pin pitch 5.00mm  length 7mm width 2.5mm Capacitor")
@@
 		(attr through_hole)
 		(fp_line
-			(start 23.6 5)
-			(end 22.8 5)
+			(start 13 5)
+			(end 12.2 5)
 			(stroke
 				(width 0.12)
@@
 		)
 		(fp_line
-			(start 23.5 0)
-			(end 22.8 0)
+			(start 12.9 0)
+			(end 12.2 0)
 			(stroke
 				(width 0.12)
@@
 		)
 		(fp_line
-			(start 22.82 6.62)
-			(end 22.82 -1.62)
+			(start 12.22 6.62)
+			(end 12.22 -1.62)
 			(stroke
 				(width 0.12)
@@
 		)
 		(fp_line
-			(start 22.82 -1.62)
+			(start 12.22 -1.62)
 			(end 2.58 -1.62)
 			(stroke
@@
 		)
 		(fp_line
-			(start 2.58 6.62)
-			(end 22.82 6.62)
+			(start 2.58 -1.62)
+			(end 2.58 6.62)
 			(stroke
 				(width 0.12)
@@
 		)
 		(fp_line
-			(start 2.58 -1.62)
-			(end 2.58 6.62)
+			(start 2 10)
+			(end 1.2 10)
 			(stroke
 				(width 0.12)
@@
 		)
 		(fp_line
-			(start 2 5)
-			(end 1.2 5)
+			(start 2 0)
+			(end 1.2 0)
 			(stroke
 				(width 0.12)
@@
 		)
 		(fp_line
-			(start 2 0)
-			(end 1.2 0)
+			(start 1.44 2.5)
+			(end 2.58 2.5)
 			(stroke
 				(width 0.12)
@@
 		)
 		(fp_line
-			(start 1.44 2.5)
-			(end 2.58 2.5)
+			(start -2.5 12.5)
+			(end 17.5 12.5)
 			(stroke
 				(width 0.12)
@@
 		)
 		(fp_line
-			(start 24.4 5)
-			(end 22.8 5)
+			(start 13.8 5)
+			(end 12.2 5)
 			(stroke
 				(width 0.1)
@@
 		)
 		(fp_line
-			(start 24.4 0)
-			(end 22.8 0)
+			(start 13.8 0)
+			(end 12.2 0)
 			(stroke
 				(width 0.1)
@@
 		)
 		(fp_line
-			(start 22.7 6.5)
-			(end 22.7 -1.5)
+			(start 12.1 6.5)
+			(end 12.1 -1.5)
 			(stroke
 				(width 0.1)
@@
 		)
 		(fp_line
-			(start 22.7 -1.5)
+			(start 12.1 -1.5)
 			(end 2.7 -1.5)
 			(stroke
@@
 		(fp_line
 			(start 2.7 6.5)
-			(end 22.7 6.5)
+			(end 12.1 6.5)
 			(stroke
 				(width 0.1)
@@
 		)
 		(fp_line
-			(start 2.6 5)
-			(end 1.2 5)
+			(start 2.6 10)
+			(end 1.2 10)
 			(stroke
 				(width 0.1)
@@
 		)
 		(pad "2" thru_hole oval
-			(at 25.4 0 180)
+			(at 15 0 180)
 			(size 2.4 2.4)
 			(drill 1.2)
@@
 		)
 		(pad "3" thru_hole circle
-			(at 0 5 180)
+			(at 0 10 180)
 			(size 2.4 2.4)
 			(drill 1.2)
@@
 		)
 		(pad "4" thru_hole oval
-			(at 25.4 5 180)
+			(at 15 10 180)
 			(size 2.4 2.4)
 			(drill 1.2)
@@
 	)
 	(segment
-		(start 91.425988 26.2)
-		(end 95.925988 30.7)
+		(start 87.45 25.475)
+		(end 89.3 25.475)
 		(width 0.6)
 		(layer "B.Cu")
@@
 	)
 	(segment
-		(start 84.1 26.2)
-		(end 91.425988 26.2)
+		(start 98.877208 29.975)
+		(end 94.377208 25.475)
 		(width 0.6)
 		(layer "B.Cu")
@@
 	)
 	(segment
-		(start 95.925988 30.7)
-		(end 96.8 30.7)
+		(start 100.15 29.975)
+		(end 98.877208 29.975)
 		(width 0.6)
 		(layer "B.Cu")
@@
 	)
 	(segment
-		(start 96.45 39.9)
-		(end 96.65 39.7)
-		(width 0.8)
-		(layer "F.Cu")
-		(net 2)
-	)
-	(segment
-		(start 96.45 39.9)
-		(end 96.65 39.7)
+		(start 94.377208 25.475)
+		(end 89.3 25.475)
 		(width 0.6)
 		(layer "B.Cu")
-		(net 2)
+		(net 1)
 	)
 	(segment
-		(start 100.6 28.35)
-		(end 98.45 26.2)
-		(width 0.6)
-		(layer "B.Cu")
+		(start 99.8 39.175)
+		(end 100 38.975)
+		(width 0.8)
+		(layer "F.Cu")
 		(net 2)
 	)
 	(segment
-		(start 98.186396 39.436396)
-		(end 100.6 37.022792)
+		(start 99.8 39.175)
+		(end 100 38.975)
 		(width 0.6)
 		(layer "B.Cu")
@@
 	)
 	(segment
-		(start 98.45 26.2)
-		(end 96.8 26.2)
+		(start 103.95 27.625)
+		(end 101.8 25.475)
 		(width 0.6)
 		(layer "B.Cu")
@@
 	)
 	(segment
-		(start 100.6 37.022792)
-		(end 100.6 28.35)
+		(start 101.536396 38.711396)
+		(end 103.95 36.297792)
 		(width 0.6)
 		(layer "B.Cu")
@@
 	)
 	(segment
-		(start 102.7 39.2)
-		(end 102.2 39.7)
+		(start 101.8 25.475)
+		(end 100.15 25.475)
 		(width 0.6)
 		(layer "B.Cu")
@@
 	)
 	(segment
-		(start 96.65 39.7)
-		(end 97.922792 39.7)
+		(start 103.95 36.297792)
+		(end 103.95 27.625)
 		(width 0.6)
 		(layer "B.Cu")
@@
 	)
 	(segment
-		(start 96.45 50.2)
-		(end 96.45 39.9)
+		(start 100 38.975)
+		(end 101.272792 38.975)
 		(width 0.6)
 		(layer "B.Cu")
@@
 	)
 	(segment
-		(start 102.2 39.7)
-		(end 97.922792 39.7)
+		(start 99.8 49.475)
+		(end 99.8 39.175)
 		(width 0.6)
 		(layer "B.Cu")
@@
 	)
 	(segment
-		(start 97.922792 39.7)
-		(end 98.186396 39.436396)
+		(start 101.272792 38.975)
+		(end 101.536396 38.711396)
 		(width 0.6)
 		(layer "B.Cu")
@@
 	)
 	(segment
+		(start 87.45 29.975)
+		(end 87.45 34.475)
+		(width 0.6)
+		(layer "B.Cu")
+		(net 3)
+	)
+	(segment
 		(start 43.95 51.8)
 		(end 43.95 44.3)
@@
 	)
 	(segment
-		(start 80.15 43.5)
-		(end 80.15 35.745)
-		(width 0.6)
-		(layer "B.Cu")
-		(net 3)
-	)
-	(segment
-		(start 80.695 35.2)
-		(end 84.1 35.2)
-		(width 0.6)
-		(layer "B.Cu")
-		(net 3)
-	)
-	(segment
-		(start 84.1 35.2)
-		(end 84.1 30.7)
+		(start 84.32 34.475)
+		(end 87.45 34.475)
 		(width 0.6)
 		(layer "B.Cu")
@@
 	)
 	(segment
-		(start 80.15 35.745)
-		(end 80.695 35.2)
+		(start 80.695 38.1)
+		(end 84.32 34.475)
 		(width 0.6)
 		(layer "B.Cu")
@@
 	)
 	(segment
-		(start 91.259084 39.7)
-		(end 83.95 39.7)
+		(start 94.609084 38.975)
+		(end 87.3 38.975)
 		(width 0.6)
 		(layer "B.Cu")
@@
 	)
 	(segment
-		(start 96.8 35.2)
-		(end 95.759084 35.2)
+		(start 100.15 34.475)
+		(end 99.109084 34.475)
 		(width 0.6)
 		(layer "B.Cu")
@@
 	)
 	(segment
-		(start 95.759084 35.2)
-		(end 91.259084 39.7)
+		(start 99.109084 34.475)
+		(end 94.609084 38.975)
 		(width 0.6)
 		(layer "B.Cu")
@@
 	)
 	(segment
-		(start 47.26 35.2)
-		(end 45.26 37.2)
-		(width 0.6)
-		(layer "B.Cu")
-		(net 5)
-	)
-	(segment
 		(start 45.26 37.2)
 		(end 41.36 41.1)
@@
 	)
 	(segment
-		(start 32.15 41.1)
-		(end 28.95 44.3)
+		(start 50.215 38.1)
+		(end 46.16 38.1)
 		(width 0.6)
 		(layer "B.Cu")
@@
 	)
 	(segment
-		(start 50.14 35.275)
-		(end 50.215 35.2)
+		(start 32.15 41.1)
+		(end 28.95 44.3)
 		(width 0.6)
 		(layer "B.Cu")
@@
 	)
 	(segment
-		(start 50.215 35.2)
-		(end 47.26 35.2)
+		(start 46.16 38.1)
+		(end 45.26 37.2)
 		(width 0.6)
 		(layer "B.Cu")

Commit message: Uploading files
Parts:
- removed C8: Capacitor_Filme, Capacitor_THT:C_Rect_L18.0mm_W6.0mm_P15.00mm_FKS3_FKP3
- added C1: Capacitor_Eletrolitico, pci:EEHZT1E331UP, F.Cu at (119.5, 96.0)
- moved U2 100.1 mm to (182.5, 117.0), turned to 90 degrees
- moved T1 95.0 mm to (132.6, 104.6)
- moved R4 90.3 mm to (161.5, 78.5)
- moved L1 89.1 mm to (162.0, 67.9)
- moved D1d4 88.0 mm to (168.1, 73.9)
- moved C3b1 88.0 mm to (124.8, 79.2)
- moved D3 88.0 mm to (126.1, 72.1)
- moved F1 88.0 mm to (118.7, 65.5)
- moved V1 88.0 mm to (111.3, 66.2)
- moved C3 88.0 mm to (132.3, 61.1)
- moved C7 88.0 mm to (169.8, 85.1)
- moved D1d1 88.0 mm to (168.3, 60.4)
- moved D1d2 88.0 mm to (168.3, 69.4)
- moved D1d3 88.0 mm to (168.3, 64.9)
- moved C10 86.1 mm to (182.0, 113.0)
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Routing:
- net Net-(D1d1-K): track 14.6 -> 25.5 mm
- net Net-(C3-Pad1): track 17.8 -> 27.4 mm
- net Net-(C3-Pad2): track 29.3 -> 37.7 mm
- net GND: track 29.3 -> 36.8 mm
- net Net-(D3-K): track 32.1 -> 28.3 mm
- net Net-(F1-Pad1): track 7.73 -> 5.73 mm
- net /BarP: track 68.4 -> 70.1 mm
Other:
- board size 80 x 60 mm -> 80 x 80 mm
