File: switched_power_supply/switched_power_supply.kicad_pcb (KiCad board)
At the start: 2 copper layers, 80 x 80 mm, 41 parts, among them IC1 VIPER53ESPTR-E, T1 Transformador_1x2, U2 TL431, U3 PC817 Opto

Commit message: atualização final
Parts:
- moved D3 0.72 mm to (118.7, 82.0)
Routing:
- net Net-(D3-K): track 28.6 -> 30.6 mm
- net GND: track 145.6 -> 146.5 mm
- net Terra: vias 1 -> 0
Other:
- board text removed: "adicionar rasgo de isolamento ou espacamento de 8mm furo pra fixar deixar trilhas com 2.5mm de distancia no primario"
Changed lines of the file:
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@@
 		(pcbplotparams
 			(layerselection 0x00010fc_ffffffff)
-			(plot_on_all_layers_selection 0x0000000_00000000)
+			(plot_on_all_layers_selection 0x0000000_80000000)
 			(disableapertmacros no)
 			(usegerberextensions no)
@@
 			(viasonmask no)
 			(mode 1)
-			(useauxorigin no)
+			(useauxorigin yes)
 			(hpglpennumber 1)
 			(hpglpenspeed 20)
@@
 			(outputformat 1)
 			(mirror no)
-			(drillshape 1)
+			(drillshape 0)
 			(scaleselection 1)
 			(outputdirectory "")
@@
 		(tags "Capacitor Polarised")
 		(property "Reference" "C9"
-			(at -7.65 9.55 180)
+			(at -7.65 9.55 0)
 			(layer "F.SilkS")
 			(effects
@@
 		(attr smd)
 		(fp_line
+			(start -3.5 6.75)
+			(end 3.5 6.75)
+			(stroke
+				(width 0.2)
+				(type default)
+			)
+			(layer "F.SilkS")
+		)
+		(fp_line
+			(start 3.5 6.75)
+			(end 6.75 3.5)
+			(stroke
+				(width 0.2)
+				(type default)
+			)
+			(layer "F.SilkS")
+		)
+		(fp_line
+			(start -6.75 3.5)
+			(end -3.5 6.75)
+			(stroke
+				(width 0.2)
+				(type default)
+			)
+			(layer "F.SilkS")
+		)
+		(fp_line
 			(start -6.75 3.5)
 			(end -6.75 -6.75)
@@
 		)
 		(fp_text user "${REFERENCE}"
-			(at -8.55 -4.075 180)
+			(at -8.55 -4.075 0)
 			(layer "F.Fab")
 			(effects
@@
 			(at 0 -3.75 0)
 			(layer "F.SilkS")
+			(hide yes)
 			(effects
 				(font
@@
 			(at 0 -3.75 0)
 			(layer "F.SilkS")
+			(hide yes)
 			(effects
 				(font
@@
 			(at 0 -3.75 0)
 			(layer "F.SilkS")
+			(hide yes)
 			(effects
 				(font
@@
 			(at 0 -3.75 0)
 			(layer "F.SilkS")
+			(hide yes)
 			(effects
 				(font
@@
 		(tags "Inductor")
 		(property "Reference" "L2"
-			(at 7.338 4.554 180)
+			(at 7.338 4.554 0)
 			(layer "F.SilkS")
 			(effects
@@
 		)
 		(property "Value" "Indutor 10uH"
-			(at 0 0 90)
+			(at 0 -3 90)
 			(layer "F.SilkS")
 			(hide yes)
@@
 		)
 		(property "Footprint" "pci:INDPM108102X400N"
-			(at 0 0 90)
+			(at 0 6.5 90)
 			(layer "F.Fab")
 			(hide yes)
@@
 		)
 		(property "Description" "Indutor"
-			(at 0 0 90)
+			(at 0 3.25 90)
 			(layer "F.Fab")
 			(hide yes)
@@
 		)
 		(fp_line
+			(start -2.5 0)
+			(end -2.75 0)
+			(stroke
+				(width 0.1)
+				(type default)
+			)
+			(layer "F.SilkS")
+		)
+		(fp_line
+			(start -2.25 0)
+			(end -2.5 0)
+			(stroke
+				(width 0.1)
+				(type default)
+			)
+			(layer "F.SilkS")
+		)
+		(fp_line
+			(start 2.25 0)
+			(end 2.75 0)
+			(stroke
+				(width 0.1)
+				(type default)
+			)
+			(layer "F.SilkS")
+		)
+		(fp_line
 			(start 5.398 -5.08)
 			(end -5.398 -5.08)
@@
 			(layer "F.SilkS")
 		)
+		(fp_arc
+			(start -2.25 0)
+			(mid -1.5 -0.75)
+			(end -0.75 0)
+			(stroke
+				(width 0.1)
+				(type default)
+			)
+			(layer "F.SilkS")
+		)
+		(fp_arc
+			(start -0.75 0)
+			(mid 0 -0.75)
+			(end 0.75 0)
+			(stroke
+				(width 0.1)
+				(type default)
+			)
+			(layer "F.SilkS")
+		)
+		(fp_arc
+			(start 0.75 0)
+			(mid 1.5 -0.75)
+			(end 2.25 0)
+			(stroke
+				(width 0.1)
+				(type default)
+			)
+			(layer "F.SilkS")
+		)
+		(fp_circle
+			(center -2 -1.25)
+			(end -1.75 -1.25)
+			(stroke
+				(width 0.1)
+				(type default)
+			)
+			(fill none)
+			(layer "F.SilkS")
+		)
 		(fp_line
 			(start -6.275 5.394)
@@
 		)
 		(fp_text user "${REFERENCE}"
-			(at 0 0 90)
+			(at 0 -6.5 90)
 			(layer "F.Fab")
 			(effects
@@
 	(footprint "Diode_THT:D_DO-41_SOD81_P7.62mm_Horizontal"
 		(layer "F.Cu")
-		(at 118.745 81.28)
+		(at 118.745 82)
 		(descr "Diode, DO-41_SOD81 series, Axial, Horizontal, pin pitch=7.62mm, , length*diameter=5.2*2.7mm^2, , http://www.diodes.com/_files/packages/DO-41%20(Plastic).pdf")
 		(tags "Diode DO-41_SOD81 series Axial Horizontal pin pitch 7.62mm  length 5.2mm diameter 2.7mm")
@@
 		)
 	)
-	(gr_text "127-220V ~ 60Hz\n"
-		(at 157 52 0)
+	(gr_text "127-220V \n~ 60Hz\n"
+		(at 113.99 58.07 0)
 		(layer "F.SilkS")
 		(effects
@@
 		)
 	)
-	(gr_text "adicionar rasgo de isolamento ou espacamento de 8mm\nfuro pra fixar\ndeixar trilhas com 2.5mm de distancia no primario\n"
-		(at 109.88 137.61 0)
-		(layer "F.SilkS")
-		(effects
-			(font
-				(size 1.5 1.5)
-				(thickness 0.3)
-				(bold yes)
-			)
-			(justify left bottom)
-		)
-	)
 	(gr_text "12VDC @ 2A"
 		(at 163.5 127.5 0)
@@
 	)
 	(segment
-		(start 135.0662 90.3)
+		(start 133.1466 92.9434)
 		(end 132.4228 92.9434)
 		(width 0.6)
@@
 	)
 	(segment
-		(start 123.8023 107.72)
-		(end 124.850257 107.72)
+		(start 142.75 89.88)
+		(end 136.21 89.88)
 		(width 0.6)
 		(layer "F.Cu")
@@
 	)
 	(segment
-		(start 134.2578 94.7784)
-		(end 132.4228 92.9434)
+		(start 146.304 86.326)
+		(end 142.75 89.88)
 		(width 0.6)
 		(layer "F.Cu")
@@
 	)
 	(segment
-		(start 134.2578 98.312457)
-		(end 134.2578 94.7784)
+		(start 123.8023 107.72)
+		(end 124.850257 107.72)
 		(width 0.6)
 		(layer "F.Cu")
@@
 	)
 	(segment
-		(start 140.8925 90.3)
-		(end 135.0662 90.3)
+		(start 134.2578 94.7784)
+		(end 132.4228 92.9434)
 		(width 0.6)
 		(layer "F.Cu")
@@
 	)
 	(segment
-		(start 116.0398 102.2434)
-		(end 116.0398 100.8634)
+		(start 134.2578 98.312457)
+		(end 134.2578 94.7784)
 		(width 0.6)
 		(layer "F.Cu")
@@
 	)
 	(segment
-		(start 146.304 84.8885)
-		(end 140.8925 90.3)
+		(start 116.0398 102.2434)
+		(end 116.0398 100.8634)
 		(width 0.6)
 		(layer "F.Cu")
@@
 	)
 	(segment
+		(start 136.21 89.88)
+		(end 133.1466 92.9434)
+		(width 0.6)
+		(layer "F.Cu")
+		(net 2)
+	)
+	(segment
 		(start 123.8023 108.164546)
 		(end 123.8023 107.72)
@@
 	)
 	(segment
+		(start 146.304 84.8885)
+		(end 146.304 86.326)
+		(width 0.6)
+		(layer "F.Cu")
+		(net 2)
+	)
+	(segment
 		(start 129.110128 103.460128)
 		(end 128.596856 103.9734)
@@
 	)
 	(segment
-		(start 114.75 78.5)
+		(start 117.125 80.875)
 		(end 117.53 81.28)
 		(width 0.6)
@@
 	)
 	(segment
+		(start 114.75 78.5)
+		(end 117.125 80.875)
+		(width 0.6)
+		(layer "B.Cu")
+		(net 5)
+	)
+	(segment
+		(start 118.25 82)
+		(end 118.745 82)
+		(width 0.6)
+		(layer "B.Cu")
+		(net 5)
+	)
+	(segment
+		(start 117.125 80.875)
+		(end 118.25 82)
+		(width 0.6)
+		(layer "B.Cu")
+		(net 5)
+	)
+	(segment
 		(start 122.4 92)
 		(end 122.4 98.2932)
@@
 	)
 	(segment
-		(start 122.4 83.1)
-		(end 122.4 92)
+		(start 137.692468 82.692467)
+		(end 139.546435 80.8385)
 		(width 0.6)
 		(layer "B.Cu")
@@
 	)
 	(segment
-		(start 126.365 81.28)
-		(end 126.935 80.71)
+		(start 149.6985 80.8385)
+		(end 151.384 82.524)
 		(width 0.6)
 		(layer "B.Cu")
@@
 	)
 	(segment
-		(start 124.22 81.28)
-		(end 122.4 83.1)
+		(start 126.365 82)
+		(end 127.057467 82.692467)
 		(width 0.6)
 		(layer "B.Cu")
@@
 	)
 	(segment
-		(start 126.935 80.71)
-		(end 149.57 80.71)
+		(start 127.057467 82.692467)
+		(end 137.692468 82.692467)
+		(width 0.6)
+		(layer "B.Cu")
+		(net 6)
+	)
+	(segment
+		(start 124.809366 82)
+		(end 122.4 84.409366)
+		(width 0.6)
+		(layer "B.Cu")
+		(net 6)
+	)
+	(segment
+		(start 126.365 82)
+		(end 124.809366 82)
+		(width 0.6)
+		(layer "B.Cu")
+		(net 6)
+	)
+	(segment
+		(start 139.546435 80.8385)
+		(end 149.6985 80.8385)
 		(width 0.6)
 		(layer "B.Cu")
@@
 	(segment
 		(start 126.365 81.28)
-		(end 124.22 81.28)
+		(end 126.835 81.75)
 		(width 0.6)
 		(layer "B.Cu")
@@
 	)
 	(segment
-		(start 149.57 80.71)
-		(end 151.384 82.524)
+		(start 122.4 84.409366)
+		(end 122.4 92)
 		(width 0.6)
 		(layer "B.Cu")
@@
 		(net 13)
 	)
-	(via
-		(at 155.1723 113.8368)
-		(size 0.6)
-		(drill 0.3)
-		(layers "F.Cu" "B.Cu")
-		(net 13)
-	)
 	(segment
 		(start 141.224 100.024)
@@
 		(min_thickness 0.25)
 		(filled_areas_thickness no)
-		(fill
+		(fill yes
 			(thermal_gap 0.5)
 			(thermal_bridge_width 0.5)
